File: tsuka60-pro-plate.kicad_sch (KiCad schematic)
At the start: 82 parts

Commit message: Finalise plate and exports
Parts:
- removed MX32, MX44: MX-NoLED, marbastlib-xp-plate-mx:Plate-MP_MX_1.75u, symbol MX_Alps_Hybrid:MX-NoLED
- removed MX65, MX71: MX-NoLED, marbastlib-xp-plate-mx:Plate-MP_MX_1.25u, symbol MX_Alps_Hybrid:MX-NoLED
- removed MX67, MX69, MX70_2: MX-NoLED, marbastlib-xp-plate-mx:Plate-MP_MX_1u, symbol MX_Alps_Hybrid:MX-NoLED
- removed S2: MX_stab, marbastlib-xp-plate-mx:Plate-MP_MX_2u, symbol marbastlib-mx:MX_stab
Changed lines of the file:
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@@
-    )
-  )
-  (global_label "44_2" (shape input) (at 217.17 133.35 180) (fields_autoplaced)
-    (effects (font (size 1.27 1.27)) (justify right))
-    (property "Intersheetrefs" "${INTERSHEET_REFS}" (at 210.1607 133.2706 0)
-      (effects (font (size 1.27 1.27)) (justify right) hide)
     )
   )
@@
     )
   )
-  (global_label "70_2" (shape input) (at 179.07 260.35 180) (fields_autoplaced)
-    (effects (font (size 1.27 1.27)) (justify right))
-    (property "Intersheetrefs" "${INTERSHEET_REFS}" (at 172.0607 260.2706 0)
-      (effects (font (size 1.27 1.27)) (justify right) hide)
-    )
-  )
   (global_label "70_2" (shape input) (at 166.37 209.55 180) (fields_autoplaced)
     (effects (font (size 1.27 1.27)) (justify right))
@@
     )
   )
-  (global_label "32_2" (shape input) (at 64.77 133.35 180) (fields_autoplaced)
-    (effects (font (size 1.27 1.27)) (justify right))
-    (property "Intersheetrefs" "${INTERSHEET_REFS}" (at 57.7607 133.2706 0)
-      (effects (font (size 1.27 1.27)) (justify right) hide)
-    )
-  )
   (global_label "COL13" (shape input) (at 158.75 255.27 270) (fields_autoplaced)
     (effects (font (size 1.27 1.27)) (justify right))
@@
     )
   )
-  (global_label "COL9" (shape input) (at 184.15 255.27 270) (fields_autoplaced)
-    (effects (font (size 1.27 1.27)) (justify right))
-    (property "Intersheetrefs" "${INTERSHEET_REFS}" (at 184.0706 262.5212 90)
-      (effects (font (size 1.27 1.27)) (justify right) hide)
-    )
-  )
   (symbol (lib_id "MX_Alps_Hybrid:MX-NoLED") (at 167.64 91.44 0) (unit 1)
     (in_bom yes) (on_board yes) (dnp no) (fields_autoplaced)
@@
         (path "/b3baaebd-c99d-4218-99ba-d40a73031965"
           (reference "MX64") (unit 1)
-        )
-      )
-    )
-  )
-  (symbol (lib_id "MX_Alps_Hybrid:MX-NoLED") (at 180.34 205.74 0) (unit 1)
-    (in_bom yes) (on_board yes) (dnp no) (fields_autoplaced)
-    (property "Reference" "MX71" (at 181.2256 199.39 0)
-      (effects (font (size 1.524 1.524)))
-    )
-    (property "Value" "MX-NoLED" (at 181.2256 200.66 0)
-      (effects (font (size 0.508 0.508)))
-    )
-    (property "Footprint" "marbastlib-xp-plate-mx:Plate-MP_MX_1.25u" (at 164.465 206.375 0)
-      (effects (font (size 1.524 1.524)) hide)
-    )
-    (property "Datasheet" "" (at 164.465 206.375 0)
-      (effects (font (size 1.524 1.524)) hide)
-    )
-    (pin "1")
-    (pin "2")
-    (instances
-      (project "tsuka60-pro-plate"
-        (path "/b3baaebd-c99d-4218-99ba-d40a73031965"
-          (reference "MX71") (unit 1)
         )
       )
@@
     )
   )
-  (symbol (lib_id "marbastlib-mx:MX_stab") (at 139.7 241.3 0) (unit 1)
-    (in_bom yes) (on_board yes) (dnp no)
-    (property "Reference" "S2" (at 138.43 245.11 0)
-      (effects (font (size 1.27 1.27)) (justify left))
-    )
-    (property "Value" "MX_stab" (at 135.89 247.65 0)
-      (effects (font (size 1.27 1.27)) (justify left))
-    )
-    (property "Footprint" "marbastlib-xp-plate-mx:Plate-MP_MX_2u" (at 139.7 241.3 0)
-      (effects (font (size 1.27 1.27)) hide)
-    )
-    (property "Datasheet" "" (at 139.7 241.3 0)
-      (effects (font (size 1.27 1.27)) hide)
-    )
-    (instances
-      (project "tsuka60-pro-plate"
-        (path "/b3baaebd-c99d-4218-99ba-d40a73031965"
-          (reference "S2") (unit 1)
-        )
-      )
-    )
-  )
   (symbol (lib_id "Mechanical:MountingHole") (at 190.5 228.6 0) (unit 1)
     (in_bom yes) (on_board yes) (dnp no) (fields_autoplaced)
@@
     )
   )
-  (symbol (lib_id "MX_Alps_Hybrid:MX-NoLED") (at 66.04 129.54 0) (unit 1)
-    (in_bom yes) (on_board yes) (dnp no) (fields_autoplaced)
-    (property "Reference" "MX32" (at 66.9256 123.19 0)
-      (effects (font (size 1.524 1.524)))
-    )
-    (property "Value" "MX-NoLED" (at 66.9256 124.46 0)
-      (effects (font (size 0.508 0.508)))
-    )
-    (property "Footprint" "marbastlib-xp-plate-mx:Plate-MP_MX_1.75u" (at 50.165 130.175 0)
-      (effects (font (size 1.524 1.524)) hide)
-    )
-    (property "Datasheet" "" (at 50.165 130.175 0)
-      (effects (font (size 1.524 1.524)) hide)
-    )
-    (pin "1")
-    (pin "2")
-    (instances
-      (project "tsuka60-pro-plate"
-        (path "/b3baaebd-c99d-4218-99ba-d40a73031965"
-          (reference "MX32") (unit 1)
-        )
-      )
-    )
-  )
   (symbol (lib_id "MX_Alps_Hybrid:MX-NoLED") (at 116.84 91.44 0) (unit 1)
     (in_bom yes) (on_board yes) (dnp no) (fields_autoplaced)
@@
     )
   )
-  (symbol (lib_id "MX_Alps_Hybrid:MX-NoLED") (at 218.44 129.54 0) (unit 1)
-    (in_bom yes) (on_board yes) (dnp no) (fields_autoplaced)
-    (property "Reference" "MX44" (at 219.3256 123.19 0)
-      (effects (font (size 1.524 1.524)))
-    )
-    (property "Value" "MX-NoLED" (at 219.3256 124.46 0)
-      (effects (font (size 0.508 0.508)))
-    )
-    (property "Footprint" "marbastlib-xp-plate-mx:Plate-MP_MX_1.75u" (at 202.565 130.175 0)
-      (effects (font (size 1.524 1.524)) hide)
-    )
-    (property "Datasheet" "" (at 202.565 130.175 0)
-      (effects (font (size 1.524 1.524)) hide)
-    )
-    (pin "1")
-    (pin "2")
-    (instances
-      (project "tsuka60-pro-plate"
-        (path "/b3baaebd-c99d-4218-99ba-d40a73031965"
-          (reference "MX44") (unit 1)
-        )
-      )
-    )
-  )
   (symbol (lib_id "MX_Alps_Hybrid:MX-NoLED") (at 205.74 205.74 0) (unit 1)
     (in_bom yes) (on_board yes) (dnp no) (fields_autoplaced)
@@
     )
   )
-  (symbol (lib_id "MX_Alps_Hybrid:MX-NoLED") (at 180.34 256.54 0) (unit 1)
-    (in_bom yes) (on_board yes) (dnp no) (fields_autoplaced)
-    (property "Reference" "MX70_2" (at 181.2256 250.19 0)
-      (effects (font (size 1.524 1.524)))
-    )
-    (property "Value" "MX-NoLED" (at 181.2256 251.46 0)
-      (effects (font (size 0.508 0.508)))
-    )
-    (property "Footprint" "marbastlib-xp-plate-mx:Plate-MP_MX_1u" (at 164.465 257.175 0)
-      (effects (font (size 1.524 1.524)) hide)
-    )
-    (property "Datasheet" "" (at 164.465 257.175 0)
-      (effects (font (size 1.524 1.524)) hide)
-    )
-    (pin "1")
-    (pin "2")
-    (instances
-      (project "tsuka60-pro-plate"
-        (path "/b3baaebd-c99d-4218-99ba-d40a73031965"
-          (reference "MX70_2") (unit 1)
-        )
-      )
-    )
-  )
   (symbol (lib_id "MX_Alps_Hybrid:MX-NoLED") (at 167.64 53.34 0) (unit 1)
     (in_bom yes) (on_board yes) (dnp no) (fields_autoplaced)
@@
         (path "/b3baaebd-c99d-4218-99ba-d40a73031965"
           (reference "MX57") (unit 1)
-        )
-      )
-    )
-  )
-  (symbol (lib_id "MX_Alps_Hybrid:MX-NoLED") (at 154.94 205.74 0) (unit 1)
-    (in_bom yes) (on_board yes) (dnp no) (fields_autoplaced)
-    (property "Reference" "MX69" (at 155.8256 199.39 0)
-      (effects (font (size 1.524 1.524)))
-    )
-    (property "Value" "MX-NoLED" (at 155.8256 200.66 0)
-      (effects (font (size 0.508 0.508)))
-    )
-    (property "Footprint" "marbastlib-xp-plate-mx:Plate-MP_MX_1u" (at 139.065 206.375 0)
-      (effects (font (size 1.524 1.524)) hide)
-    )
-    (property "Datasheet" "" (at 139.065 206.375 0)
-      (effects (font (size 1.524 1.524)) hide)
-    )
-    (pin "1")
-    (pin "2")
-    (instances
-      (project "tsuka60-pro-plate"
-        (path "/b3baaebd-c99d-4218-99ba-d40a73031965"
-          (reference "MX69") (unit 1)
         )
       )
@@
     )
   )
-  (symbol (lib_id "MX_Alps_Hybrid:MX-NoLED") (at 129.54 205.74 0) (unit 1)
-    (in_bom yes) (on_board yes) (dnp no) (fields_autoplaced)
-    (property "Reference" "MX67" (at 130.4256 199.39 0)
-      (effects (font (size 1.524 1.524)))
-    )
-    (property "Value" "MX-NoLED" (at 130.4256 200.66 0)
-      (effects (font (size 0.508 0.508)))
-    )
-    (property "Footprint" "marbastlib-xp-plate-mx:Plate-MP_MX_1u" (at 113.665 206.375 0)
-      (effects (font (size 1.524 1.524)) hide)
-    )
-    (property "Datasheet" "" (at 113.665 206.375 0)
-      (effects (font (size 1.524 1.524)) hide)
-    )
-    (pin "1")
-    (pin "2")
-    (instances
-      (project "tsuka60-pro-plate"
-        (path "/b3baaebd-c99d-4218-99ba-d40a73031965"
-          (reference "MX67") (unit 1)
-        )
-      )
-    )
-  )
   (symbol (lib_id "MX_Alps_Hybrid:MX-NoLED") (at 66.04 167.64 0) (unit 1)
     (in_bom yes) (on_board yes) (dnp no) (fields_autoplaced)
@@
         )
       )
-    )
-  )
-  (symbol (lib_id "MX_Alps_Hybrid:MX-NoLED") (at 104.14 205.74 0) (unit 1)
-    (in_bom yes) (on_board yes) (dnp no) (fields_autoplaced)
-    (property "Reference" "MX65" (at 105.0256 199.39 0)
-      (effects (font (size 1.524 1.524)))
-    )
-    (property "Value" "MX-NoLED" (at 105.0256 200.66 0)
-      (effects (font (size 0.508 0.508)))
-    )
-    (property "Footprint" "marbastlib-xp-plate-mx:Plate-MP_MX_1.25u" (at 88.265 206.375 0)
-      (effects (font (size 1.524 1.524)) hide)
-    )
-    (property "Datasheet" "" (at 88.265 206.375 0)
-      (effects (font (size 1.524 1.524)) hide)
-    )
-    (pin "1")
-    (pin "2")
-    (instances
-      (project "tsuka60-pro-plate"
-        (path "/b3baaebd-c99d-4218-99ba-d40a73031965"
-          (reference "MX65") (unit 1)
-        )
-      )

Commit message: Adjust standoff footprint and correct orientation, produce production files
Parts:
- H1, H2, H3, H4, H5, H6: footprint MountingHole:MountingHole_2.2mm_M2_Pad_TopOnly -> MountingHole:MountingHole_2.5mm_Pad_TopOnly
